Commit message: add fast lio and lidar 3d

File: src/ttbot_description/urdf/ttbot.urdf.xacro (robot description, xacro)
@@ -182,4 +182,33 @@
     </inertial>
   </link>
+  <!-- ================= LIDAR LINK ================= -->
+  <link name="lidar_link">
+    <visual>
+      <origin xyz="0 0 0" rpy="0 0 0"/>
+      <geometry>
+        <cylinder radius="0.05" length="0.07"/>
+      </geometry>
+      <material name="lidar_blue">
+        <color rgba="0 0 1 1"/>
+      </material>
+    </visual>
+    <collision>
+      <origin xyz="0 0 0" rpy="0 0 0"/>
+      <geometry>
+        <cylinder radius="0.05" length="0.07"/>
+      </geometry>
+    </collision>
+    <inertial>
+      <mass value="0.1"/>
+      <origin xyz="0 0 0" rpy="0 0 0"/>
+      <inertia ixx="0.0001" ixy="0" ixz="0" iyy="0.0001" iyz="0" izz="0.0001"/>
+    </inertial>
+  </link>
+  <!-- ================= LIDAR JOINT ================= -->
+  <joint name="lidar_joint" type="fixed">
+    <parent link="base_link"/>
+    <child link="lidar_link"/>
+    <origin xyz="0 0 ${wheel_radius + chassis_height + 0.2}" rpy="0 0 0"/>
+  </joint>
   <!-- ================= IMU JOINT ================= -->
   <joint name="imu_joint" type="fixed">

File: src/ttbot_description/urdf/ttbot_gazebo.xacro (robot description, xacro)
@@ -112,4 +112,41 @@
     </sensor>
   </gazebo>
+  <gazebo reference="lidar_link">
+      <sensor name="velodyne_vlp16" type="gpu_lidar">
+          <pose>0 0 0 0 0 0</pose>
+          <topic>/velodyne_points</topic>  <!-- Add leading / -->
+          <ignition_frame_id>lidar_link</ignition_frame_id>  <!-- Add this -->
+          <update_rate>10</update_rate>
+          <gz_frame_id>lidar_link</gz_frame_id>
+          <visualize>true</visualize>
+          <always_on>true</always_on>
+          <ray>
+              <scan>
+                <horizontal>
+                  <samples>1000</samples>
+                  <resolution>1</resolution>
+                  <min_angle>-3.14159265359</min_angle>
+                  <max_angle>3.14159265359</max_angle>
+                </horizontal>
+                <vertical>
+                  <samples>16</samples>
+                  <resolution>1</resolution>
+                  <min_angle>-0.261799</min_angle>
+                  <max_angle>0.261799</max_angle>
+                </vertical>
+              </scan>
+              <range>
+                  <min>0.3</min>
+                  <max>100.0</max>
+                  <resolution>0.01</resolution>
+              </range>
+              <noise>
+                  <type>gaussian</type>
+                  <mean>0.0</mean>
+                  <stddev>0.01</stddev>
+              </noise>
+          </ray>
+      </sensor>
+  </gazebo>
   <gazebo>
       <plugin filename="ignition-gazebo-navsat-system"

Commit message: resize transform

File: src/ttbot_description/urdf/ttbot.urdf.xacro (robot description, xacro)
@@ -4,10 +4,10 @@
   <xacro:include filename="$(find ttbot_description)/urdf/ttbot_gazebo.xacro" />
   <xacro:property name="wheel_radius" value="0.15"/>
-  <xacro:property name="wheel_width"  value="0.06"/>
+  <xacro:property name="wheel_width"  value="0.11"/>
   <xacro:property name="wheelbase"    value="0.65"/>
   <xacro:property name="track_width"  value="0.55"/>
   <xacro:property name="chassis_length" value="1.0"/>
-  <xacro:property name="chassis_width"  value="0.6"/>
-  <xacro:property name="chassis_height" value="0.45"/>
+  <xacro:property name="chassis_width"  value="0.55"/>
+  <xacro:property name="chassis_height" value="0.25"/>
   <xacro:macro name="inertial_cyl" params="mass r l">
     <inertial>

Commit message: add log sensor data

File: src/ttbot_description/urdf/ttbot.urdf.xacro (robot description, xacro)
@@ -209,5 +209,5 @@
     <parent link="base_link"/>
     <child link="lidar_link"/>
-    <origin xyz="-0.30 -0.03 1.50" rpy="0 0 0"/>
+    <origin xyz="-0.23 -0.03 1.47" rpy="0 0 0"/>
   </joint>
   <!-- ================= IMU JOINT ================= -->
@@ -215,5 +215,5 @@
     <parent link="base_link"/>
     <child link="imu_link"/>
-    <origin xyz="-0.20 -0.03 1.50" rpy="0 0 0"/>
+    <origin xyz="-0.20 -0.03 1.38" rpy="0 0 0"/>
   </joint>
   <!-- ================= GPS LINK ================= -->
@@ -271,5 +271,5 @@
     <parent link="base_link"/>
     <child link="camera_link"/>
-    <origin xyz="-0.20 -0.05 1.46" rpy="0 0 0"/>
+    <origin xyz="-0.12 -0.03 1.38" rpy="0 0 0"/>
   </joint>
   <link name="camera_color_optical_frame"></link>

Commit message: add pcd2pgm, fastlio pub map, nav2, new a*

File: src/ttbot_description/urdf/ttbot.urdf.xacro (robot description, xacro)
@@ -309,4 +309,12 @@
       <state_interface name="velocity"/>
     </joint>
+    <joint name="front_left_wheel_joint">
+      <state_interface name="position"/>
+      <state_interface name="velocity"/>
+    </joint>
+    <joint name="front_right_wheel_joint">
+      <state_interface name="position"/>
+      <state_interface name="velocity"/>
+    </joint>
   </ros2_control>
   <xacro:ttbot_gazebo/>
